File: _Eagle/v2/pogo board 2034.brd (EAGLE design)
At the start: 21 x 13.8 mm, 6 parts

Commit message: edit 2034
Parts:
- moved U$1 6.00 mm to (7.50, 2.38)
- moved U$2 6.00 mm to (13.5, 2.38)
Routing:
- net N$3: track 11.7 -> 23.4 mm, vias 7 -> 10
- net N$1: track 10.0 -> 0.00 mm, vias 7 -> 0
- removed copper zone on layer 16, net N$1
